File: Hardware/hymRC/hymRC.sch (KiCad schematic (older format))
At the start: 206 parts, among them J1 Relay_0, J10 EXT_AUD_IN, J11 EXT_AUD_OUT, J2 Digital Sensor Connector, J3 Analog Sensor Connector, J4 TX RADIO, J5 RX RADIO, J6 Relay_1, J7 Relay_2, J8 Relay_3, J9 Relay_4, K1 Role, K2 Role, K3 Role, K4 Role, K5 Role, Q1 BC817, Q2 NPN, Q3 NPN, Q4 NPN, Q5 NPN, U1 KT8870, U10 OptoCoupler, U11 OptoCoupler, U12 OptoCoupler, U13 OptoCoupler, U14 OptoCoupler, U2 MCP23017_SP, U3 OptoCoupler, U4 OptoCoupler, U5 OptoCoupler, U6 TL084, U7 TL084, U8 LM7808_TO220, U9 L7805, Y1 3.5795M

Commit message: initial PCB
Parts:
- D1, D2, D3, D4: footprint (none) -> Diode_SMD:D_0805_2012Metric_Pad1.15x1.40mm_HandSolder
- D5: renamed from D7; footprint (none) -> Diode_SMD:D_0805_2012Metric_Pad1.15x1.40mm_HandSolder
- J10, J11: footprint (none) -> TerminalBlock:TerminalBlock_bornier-2_P5.08mm
- J2, J3: footprint (none) -> TerminalBlock_4Ucon:TerminalBlock_4Ucon_1x09_P3.50mm_Horizontal
- R32, R46, R47: value 91K -> 100K; footprint (none) -> Resistor_SMD:R_0805_2012Metric_Pad1.20x1.40mm_HandSolder
- R34, R36, R37, R38, R39, R48, R49, R50, R51, R52, R53, R54, R55, R56, R57, R58, R59, R60, R61, R62, R63, R64, R65: footprint (none) -> Resistor_SMD:R_0805_2012Metric_Pad1.20x1.40mm_HandSolder
- RV1, RV2, RV3, RV4, RV5, RV6, RV7, RV8: footprint (none) -> Potentiometer_SMD:Potentiometer_ACP_CA9-VSMD_Vertical
- U9: footprint (none) -> Package_TO_SOT_THT:TO-220-3_Vertical
- Y1: footprint (none) -> Crystal:Crystal_SMD_SeikoEpson_MC405-2Pin_9.6x4.1mm_HandSoldering
- renumbered D5 to D7

Commit message: Audio section completed
Parts:
- K1, K2, K3: symbol hymRC_components:Role-1 -> hymRC-rescue:Role-1-hymRC_components
Connections:
- net +12V: now also C40.2, C41.2, C42.1, C43.1
- net GND: now also C40.1, C41.1, C42.2, C43.2
Changed lines of the file:
@@
 $EndComp
 $Comp
-L hymRC_components:Role-1 K1
+L hymRC-rescue:Role-1-hymRC_components K1
 U 1 1 60477DC9
 P 1650 9750
@@
 $EndComp
 $Comp
-L hymRC_components:Role-1 K2
+L hymRC-rescue:Role-1-hymRC_components K2
 U 1 1 604D7A49
 P 3400 9700
@@
 $EndComp
 $Comp
-L hymRC_components:Role-1 K3
+L hymRC-rescue:Role-1-hymRC_components K3
 U 1 1 6050AB0C
 P 5100 9700
@@
 L power:GND #PWR060
 U 1 1 611A9AB4
-P 1150 5850
-F 0 "#PWR060" H 1150 5600 50  0001 C CNN
-F 1 "GND" H 1155 5677 50  0000 C CNN
-F 2 "" H 1150 5850 50  0001 C CNN
-F 3 "" H 1150 5850 50  0001 C CNN
-	1    1150 5850
+P 1150 5900
+F 0 "#PWR060" H 1150 5650 50  0001 C CNN
+F 1 "GND" H 1155 5727 50  0000 C CNN
+F 2 "" H 1150 5900 50  0001 C CNN
+F 3 "" H 1150 5900 50  0001 C CNN
+	1    1150 5900
 	1    0    0    -1
 $EndComp
@@
 $Comp
 L hymRC_components:TL084 U6
-U 5 1 611A9A22
-P 1250 5550
-F 0 "U6" H 1208 5596 50  0000 L CNN
-F 1 "TL084" H 1208 5505 50  0000 L CNN
-F 2 "Package_SO:SOIC-14_3.9x8.7mm_P1.27mm" H 1200 5650 50  0001 C CNN
-F 3 "https://pdf.direnc.net/upload/tl081-tl082-tl084-datasheet.pdf" H 1300 5750 50  0001 C CNN
-F 4 "https://bluemavi.com/vitrin/tablo_new.asp?adet=1&kitap_id=758504#ara" H 1250 5550 50  0001 C CNN "bluemavi"
-F 5 "https://www.digikey.com/en/products/detail/texas-instruments/TL084BCD/476131" H 1250 5550 50  0001 C CNN "digikey"
-F 6 "https://www.direnc.net/tl084-smd-jfet-input-operational-amplifiers" H 1250 5550 50  0001 C CNN "direnc.net"
-F 7 "2TL" H 1250 5550 50  0001 C CNN "fiyat"
-	5    1250 5550
-	1    0    0    -1
-$EndComp
-$Comp
-L hymRC_components:TL084 U6
 U 4 1 611A9A1C
 P 2450 6500
@@
 	1    0    0    -1
 $EndComp
-Text GLabel 1150 1900 1    50   Input ~ 0
+Text GLabel 1150 1850 1    50   Input ~ 0
 Aku_12V
 Text Label 1650 1850 3    50   ~ 0
@@
 L power:GND #PWR045
 U 1 1 6080E9C6
-P 1150 2500
-F 0 "#PWR045" H 1150 2250 50  0001 C CNN
-F 1 "GND" H 1155 2327 50  0000 C CNN
-F 2 "" H 1150 2500 50  0001 C CNN
-F 3 "" H 1150 2500 50  0001 C CNN
-	1    1150 2500
+P 1150 2550
+F 0 "#PWR045" H 1150 2300 50  0001 C CNN
+F 1 "GND" H 1155 2377 50  0000 C CNN
+F 2 "" H 1150 2550 50  0001 C CNN
+F 3 "" H 1150 2550 50  0001 C CNN
+	1    1150 2550
 	1    0    0    -1
 $EndComp
@@
 $Comp
 L hymRC_components:TL084 U7
-U 5 1 60701598
-P 1250 2200
-F 0 "U7" H 1208 2246 50  0000 L CNN
-F 1 "TL084" H 1208 2155 50  0000 L CNN
-F 2 "Package_SO:SOIC-14_3.9x8.7mm_P1.27mm" H 1200 2300 50  0001 C CNN
-F 3 "https://pdf.direnc.net/upload/tl081-tl082-tl084-datasheet.pdf" H 1300 2400 50  0001 C CNN
-F 4 "https://bluemavi.com/vitrin/tablo_new.asp?adet=1&kitap_id=758504#ara" H 1250 2200 50  0001 C CNN "bluemavi"
-F 5 "https://www.digikey.com/en/products/detail/texas-instruments/TL084BCD/476131" H 1250 2200 50  0001 C CNN "digikey"
-F 6 "https://www.direnc.net/tl084-smd-jfet-input-operational-amplifiers" H 1250 2200 50  0001 C CNN "direnc.net"
-F 7 "2TL" H 1250 2200 50  0001 C CNN "fiyat"
-	5    1250 2200
-	1    0    0    -1
-$EndComp
-$Comp
-L hymRC_components:TL084 U7
 U 4 1 60700441
 P 2450 3150
@@
 	1    0    0    -1
 $EndComp
-Wire Wire Line
-	1000 2050 1000 2100
-Wire Wire Line
-	1000 2050 1550 2050
-Wire Wire Line
-	1550 2050 1550 2100
-Wire Wire Line
-	1000 2350 1000 2300
-Wire Wire Line
-	1550 2350 1550 2300
-Wire Wire Line
-	1000 2350 1550 2350
 $Comp
 L Device:C_Small C41
@@
 	1    0    0    -1
 $EndComp
-Wire Wire Line
-	1450 5400 1450 5450
-Wire Wire Line
-	1050 5400 1050 5450
-Wire Wire Line
-	1050 5400 1450 5400
-Wire Wire Line
-	1050 5700 1050 5650
-Wire Wire Line
-	1450 5700 1450 5650
-Wire Wire Line
-	1050 5700 1450 5700
 $Comp
 L Device:C_Small C45
@@
 Wire Wire Line
 	12800 4700 12800 4750
-Connection ~ 8650 7300
-Connection ~ 8800 7150
-Connection ~ 8500 7150
 $Comp
 L power:PWR_FLAG #FLG0101
@@
 	0    1    1    0
 $EndComp
+Wire Wire Line
+	1000 2100 1000 1900
+Wire Wire Line
+	1000 1900 1150 1900
+Wire Wire Line
+	1150 1900 1550 1900
+Wire Wire Line
+	1550 1900 1550 2100
+Connection ~ 1150 1900
+Wire Wire Line
+	1550 2300 1550 2500
+Wire Wire Line
+	1550 2500 1150 2500
+Wire Wire Line
+	1150 2500 1150 2550
+Connection ~ 1150 2500
+Wire Wire Line
+	1150 2500 1000 2500
+Wire Wire Line
+	1000 2500 1000 2300
+Wire Wire Line
+	1150 1850 1150 1900
+Wire Wire Line
+	1150 5250 1050 5250
+Wire Wire Line
+	1050 5250 1050 5450
+Connection ~ 1150 5250
+Wire Wire Line
+	1150 5850 1150 5900
+Wire Wire Line
+	1450 5650 1450 5850
+Wire Wire Line
+	1450 5850 1150 5850
+Connection ~ 1150 5850
+Wire Wire Line
+	1050 5650 1050 5850
+Wire Wire Line
+	1050 5850 1150 5850
+Wire Wire Line
+	1450 5250 1150 5250
+Wire Wire Line
+	1450 5250 1450 5450
+$Comp
+L hymRC_components:TL084 U6
+U 5 1 611A9A22
+P 1250 5550
+F 0 "U6" H 1208 5596 50  0000 L CNN
+F 1 "TL084" H 1208 5505 50  0000 L CNN
+F 2 "Package_SO:SOIC-14_3.9x8.7mm_P1.27mm" H 1200 5650 50  0001 C CNN
+F 3 "https://pdf.direnc.net/upload/tl081-tl082-tl084-datasheet.pdf" H 1300 5750 50  0001 C CNN
+F 4 "https://bluemavi.com/vitrin/tablo_new.asp?adet=1&kitap_id=758504#ara" H 1250 5550 50  0001 C CNN "bluemavi"
+F 5 "https://www.digikey.com/en/products/detail/texas-instruments/TL084BCD/476131" H 1250 5550 50  0001 C CNN "digikey"
+F 6 "https://www.direnc.net/tl084-smd-jfet-input-operational-amplifiers" H 1250 5550 50  0001 C CNN "direnc.net"
+F 7 "2TL" H 1250 5550 50  0001 C CNN "fiyat"
+	5    1250 5550
+	1    0    0    -1
+$EndComp
+$Comp
+L hymRC_components:TL084 U7
+U 5 1 60701598
+P 1250 2200
+F 0 "U7" H 1208 2246 50  0000 L CNN
+F 1 "TL084" H 1208 2155 50  0000 L CNN
+F 2 "Package_SO:SOIC-14_3.9x8.7mm_P1.27mm" H 1200 2300 50  0001 C CNN
+F 3 "https://pdf.direnc.net/upload/tl081-tl082-tl084-datasheet.pdf" H 1300 2400 50  0001 C CNN
+F 4 "https://bluemavi.com/vitrin/tablo_new.asp?adet=1&kitap_id=758504#ara" H 1250 2200 50  0001 C CNN "bluemavi"
+F 5 "https://www.digikey.com/en/products/detail/texas-instruments/TL084BCD/476131" H 1250 2200 50  0001 C CNN "digikey"
+F 6 "https://www.direnc.net/tl084-smd-jfet-input-operational-amplifiers" H 1250 2200 50  0001 C CNN "direnc.net"
+F 7 "2TL" H 1250 2200 50  0001 C CNN "fiyat"
+	5    1250 2200
+	1    0    0    -1
+$EndComp
 $EndSCHEMATC

Commit message: all connected somehow
Parts:
- added J12: 12V_AKU, TerminalBlock:TerminalBlock_bornier-2_P5.08mm, symbol Connector:Screw_Terminal_01x02
Connections:
- net +12V: now also J12.1 (Pin_1)
- net 5V: now also J3.5 (Pin_5); no longer J3.1 (Pin_1)
- net Analog_Sensor1: now also J3.3 (Pin_3); no longer J3.2 (Pin_2)
- net Analog_Sensor2: now also J3.4 (Pin_4); no longer J3.3 (Pin_3)
- net Digital_IN0: now also J3.8 (Pin_8); no longer J3.4 (Pin_4)
- net Digital_IN1: now also J3.7 (Pin_7); no longer J3.5 (Pin_5)
- net GND: now also J4.5 (Pin_5), J12.2 (Pin_2); no longer J4.2 (Pin_2)
- net LINK_AUDIO_IN: now also J4.6 (Pin_6); no longer J4.5 (Pin_5)
- net LINK_PTT_OUT: now also J4.3 (Pin_3); no longer J4.6 (Pin_6)
- net R0_COM: now also J1.2 (Pin_2); no longer J1.1 (Pin_1)
- net R0_NC: now also J1.3 (Pin_3); no longer J1.2 (Pin_2)
- net R1_COM: now also J6.2 (Pin_2); no longer J6.1 (Pin_1)
- net R1_NC: now also J6.3 (Pin_3); no longer J6.2 (Pin_2)
- net R1_NO: now also J6.1 (Pin_1); no longer J6.3 (Pin_3)
- net R2_COM: now also J7.2 (Pin_2); no longer J7.1 (Pin_1)
- net R2_NC: now also J7.3 (Pin_3); no longer J7.2 (Pin_2)
- net R2_NO: now also J7.1 (Pin_1); no longer J7.3 (Pin_3)
- net R3_COM1: now also J8.2 (Pin_2); no longer J8.1 (Pin_1)
- net R3_COM2: now also J8.5 (Pin_5); no longer J8.4 (Pin_4)
- net R3_NC1: now also J8.1 (Pin_1); no longer J8.2 (Pin_2)
- net R3_NC2: now also J8.4 (Pin_4); no longer J8.5 (Pin_5)
- net R4_COM1: now also J9.2 (Pin_2); no longer J9.1 (Pin_1)
- net R4_COM2: now also J9.5 (Pin_5); no longer J9.4 (Pin_4)
- net R4_NC1: now also J9.1 (Pin_1); no longer J9.2 (Pin_2)
- net R4_NC2: now also J9.4 (Pin_4); no longer J9.5 (Pin_5)
- net RO_NO: now also J1.1 (Pin_1); no longer J1.3 (Pin_3)
- net TX_AUDIO: now also J4.4 (Pin_4); no longer J4.1 (Pin_1)
- net TX_POWER: now also J4.1 (Pin_1); no longer J4.4 (Pin_4)
- net TX_PTT: now also J4.2 (Pin_2); no longer J4.3 (Pin_3)
- net UART_RX: now also J3.1 (Pin_1); no longer J3.7 (Pin_7)
- net UART_TX: now also J3.2 (Pin_2); no longer J3.8 (Pin_8)
Changed lines of the file:
@@
 Text Label 11700 1550 2    50   ~ 0
 INTA
-Text GLabel 15500 5750 0    50   Input ~ 0
+Text GLabel 15600 5750 0    50   Input ~ 0
 Digital_IN2
-Text GLabel 15500 5650 0    50   Input ~ 0
+Text GLabel 15600 5850 0    50   Input ~ 0
 Digital_IN1
-Text GLabel 15500 5550 0    50   Input ~ 0
+Text GLabel 15600 5950 0    50   Input ~ 0
 Digital_IN0
 Text GLabel 15300 9000 0    50   Input ~ 0
 R3_NO2
-Text GLabel 15300 8900 0    50   Input ~ 0
-R3_NC2
 Text GLabel 15300 8800 0    50   Input ~ 0
+R3_NC2
+Text GLabel 15300 8900 0    50   Input ~ 0
 R3_COM2
 Text GLabel 15300 8700 0    50   Input ~ 0
 R3_NO1
-Text GLabel 15300 8600 0    50   Input ~ 0
-R3_NC1
 Text GLabel 15300 8500 0    50   Input ~ 0
+R3_NC1
+Text GLabel 15300 8600 0    50   Input ~ 0
 R3_COM1
-Text GLabel 15300 8350 0    50   Input ~ 0
+Text GLabel 15300 8150 0    50   Input ~ 0
 R2_NO
-Text GLabel 15300 8250 0    50   Input ~ 0
+Text GLabel 15300 8350 0    50   Input ~ 0
 R2_NC
-Text GLabel 15300 8150 0    50   Input ~ 0
+Text GLabel 15300 8250 0    50   Input ~ 0
 R2_COM
-Text GLabel 15300 8000 0    50   Input ~ 0
+Text GLabel 15300 7800 0    50   Input ~ 0
 R1_NO
-Text GLabel 15300 7900 0    50   Input ~ 0
+Text GLabel 15300 8000 0    50   Input ~ 0
 R1_NC
-Text GLabel 15300 7800 0    50   Input ~ 0
+Text GLabel 15300 7900 0    50   Input ~ 0
 R1_COM
-Text GLabel 15300 7650 0    50   Input ~ 0
+Text GLabel 15300 7450 0    50   Input ~ 0
 RO_NO
-Text GLabel 15300 7550 0    50   Input ~ 0
+Text GLabel 15300 7650 0    50   Input ~ 0
 R0_NC
-Text GLabel 15300 7450 0    50   Input ~ 0
+Text GLabel 15300 7550 0    50   Input ~ 0
 R0_COM
 Text Notes 14650 9850 0    50   ~ 0
@@
 Wire Notes Line
 	16000 7350 16000 9900
-Text GLabel 15500 5450 0    50   Input ~ 0
+Text GLabel 15600 5550 0    50   Input ~ 0
 Analog_Sensor2
-Text GLabel 15500 5350 0    50   Input ~ 0
+Text GLabel 15600 5450 0    50   Input ~ 0
 Analog_Sensor1
 Wire Notes Line
@@
 	16000 6350 14650 6350
 Wire Wire Line
-	15600 5750 15500 5750
-Wire Wire Line
-	15600 5650 15500 5650
-Wire Wire Line
-	15600 5550 15500 5550
-Wire Wire Line
-	15600 5450 15500 5450
-Wire Wire Line
 	15600 5350 15500 5350
-Wire Wire Line
-	15500 5250 15500 5200
-Wire Wire Line
-	15600 5250 15500 5250
-Wire Wire Line
-	15500 6050 15500 6100
-Wire Wire Line
-	15600 6050 15500 6050
-$Comp
-L power:GND #PWR034
-U 1 1 60400CC3
-P 15500 6100
-F 0 "#PWR034" H 15500 5850 50  0001 C CNN
-F 1 "GND" H 15350 6050 50  0000 C CNN
-F 2 "" H 15500 6100 50  0001 C CNN
-F 3 "" H 15500 6100 50  0001 C CNN
-	1    15500 6100
-	1    0    0    -1
-$EndComp
 $Comp
 L Connector:Conn_01x09_Female J3
@@
 Text Label 15700 6650 2    50   ~ 0
 GND
-Text Label 14800 6650 2    50   ~ 0
+Text Label 14800 6950 2    50   ~ 0
 GND
-Text Label 14800 6550 2    50   ~ 0
+Text Label 14800 6850 2    50   ~ 0
 TX_AUDIO
-Text Label 14800 6750 2    50   ~ 0
+Text Label 14800 6650 2    50   ~ 0
 TX_PTT
 Text Label 15700 6850 2    50   ~ 0
@@
 	1    0    0    -1
 $EndComp
-Text Label 14800 6850 2    50   ~ 0
+Text Label 14800 6550 2    50   ~ 0
 TX_POWER
 Wire Notes Line
@@
 	1    0    0    -1
 $EndComp
-Text GLabel 15300 9150 0    50   Input ~ 0
-R4_COM1
 Text GLabel 15300 9250 0    50   Input ~ 0
+R4_COM1
+Text GLabel 15300 9150 0    50   Input ~ 0
 R4_NC1
 Text GLabel 15300 9350 0    50   Input ~ 0
 R4_NO1
-Text GLabel 15300 9450 0    50   Input ~ 0
-R4_COM2
 Text GLabel 15300 9550 0    50   Input ~ 0
+R4_COM2
+Text GLabel 15300 9450 0    50   Input ~ 0
 R4_NC2
 Text GLabel 15300 9650 0    50   Input ~ 0
@@
 Text Notes 11350 7650 0    50   ~ 0
 DIGITAL INPUT OPTOCOUPLERS
-Text Label 11550 5600 0    50   ~ 0
+Text Label 2650 6850 0    50   ~ 0
 CONTROL_INPUT_0
 $Comp
@@
 U 1 1 61D1BC7A
 P 13100 5900
-F 0 "U11" H 13100 6225 50  0000 C CNN
+F 0 "U11" H 13150 5950 50  0000 C CNN
 F 1 "OptoCoupler" H 13100 6134 50  0000 C CNN
 F 2 "Package_DIP:SMDIP-4_W7.62mm" H 13100 5550 50  0001 C CIN
@@
 	1    0    0    -1
 $EndComp
-Text Label 14800 6950 2    50   ~ 0
-LINK_AUDIO_IN
 Text Label 14800 7050 2    50   ~ 0
+LINK_AUDIO_IN
+Text Label 14800 6750 2    50   ~ 0
 LINK_PTT_OUT
 Wire Notes Line
@@
 Text Label 15500 3700 0    50   ~ 0
 5V
-Text Label 15500 5200 0    50   ~ 0
-5V
 Wire Wire Line
 	9850 1350 9850 1300
-Text GLabel 15500 5850 0    50   Input ~ 0
+Text GLabel 15500 5250 0    50   Input ~ 0
 UART_RX
-Text GLabel 15500 5950 0    50   Input ~ 0
+Text GLabel 15500 5350 0    50   Input ~ 0
 UART_TX
-Wire Wire Line
-	15600 5850 15500 5850
-Wire Wire Line
-	15600 5950 15500 5950
 Text Label 11700 1650 2    50   ~ 0
 SQUELCH
@@
 	1    0    0    -1
 $EndComp
+$Comp
+L Connector:Screw_Terminal_01x02 J12
+U 1 1 6086AFB5
+P 7550 6600
+F 0 "J12" H 7630 6592 50  0000 L CNN
+F 1 "12V_AKU" H 7630 6501 50  0000 L CNN
+F 2 "TerminalBlock:TerminalBlock_bornier-2_P5.08mm" H 7550 6600 50  0001 C CNN
+F 3 "~" H 7550 6600 50  0001 C CNN
+	1    7550 6600
+	1    0    0    -1
+$EndComp
+Text GLabel 7350 6600 0    50   Input ~ 0
+Aku_12V
+$Comp
+L power:GND #PWR07
+U 1 1 608735DD
+P 7350 6700
+F 0 "#PWR07" H 7350 6450 50  0001 C CNN
+F 1 "GND" H 7355 6527 50  0000 C CNN
+F 2 "" H 7350 6700 50  0001 C CNN
+F 3 "" H 7350 6700 50  0001 C CNN
+	1    7350 6700
+	1    0    0    -1
+$EndComp
+Text Label 11550 5600 0    50   ~ 0
+CONTROL_INPUT_0
+Wire Wire Line
+	15500 6050 15500 6100
+Wire Wire Line
+	15600 6050 15500 6050
+Wire Wire Line
+	15600 5250 15500 5250
+Text Label 15500 5650 2    50   ~ 0
+5V
+$Comp
+L power:GND #PWR034
+U 1 1 60400CC3
+P 15500 6100
+F 0 "#PWR034" H 15500 5850 50  0001 C CNN
+F 1 "GND" H 15350 6050 50  0000 C CNN
+F 2 "" H 15500 6100 50  0001 C CNN
+F 3 "" H 15500 6100 50  0001 C CNN
+	1    15500 6100
+	1    0    0    -1
+$EndComp
+Wire Wire Line
+	15600 5650 15500 5650
 $EndSCHEMATC

Commit message: digitals connected
Connections:
- net GND: now also J5.5 (Pin_5); no longer J5.2 (Pin_2)
- net LINK_SQL: now also J5.2 (Pin_2); no longer J5.5 (Pin_5)
- net RX_AUDIO: now also J5.4 (Pin_4); no longer J5.1 (Pin_1)
- net RX_SQL: now also J5.1 (Pin_1); no longer J5.4 (Pin_4)
Changed lines of the file:
@@
 Text Notes 9400 8700 0    50   ~ 0
 REGULATORS
-Text Label 15700 6550 2    50   ~ 0
+Text Label 15700 6850 2    50   ~ 0
 RX_AUDIO
-Text Label 15700 6650 2    50   ~ 0
+Text Label 15700 6950 2    50   ~ 0
 GND
 Text Label 14800 6950 2    50   ~ 0
@@
 Text Label 14800 6650 2    50   ~ 0
 TX_PTT
-Text Label 15700 6850 2    50   ~ 0
+Text Label 15700 6550 2    50   ~ 0
 RX_SQL
 $Comp
@@
 Text Label 15700 6750 2    50   ~ 0
 LINK_AUDIO_OUT
-Text Label 15700 6950 2    50   ~ 0
+Text Label 15700 6650 2    50   ~ 0
 LINK_SQL
 Text Label 11700 2250 2    50   ~ 0

Commit message: routing finished
Connections:
- net CONTROL_OUTPUT_0: now also R16.2; no longer R4.2
- net CONTROL_OUTPUT_2: now also R4.2; no longer R16.2
- net Digital_Sensor_CS1: now also J2.8 (Pin_8); no longer J2.6 (Pin_6)
- net Digital_Sensor_CS3: now also J2.6 (Pin_6); no longer J2.8 (Pin_8)
- net LINK_AUDIO_OUT: now also J5.4 (Pin_4); no longer J5.3 (Pin_3)
- net LINK_PTT_CTRL: now also A1.25 (A6); no longer A1.26 (A7)
- net RX_AUDIO: now also J5.3 (Pin_3); no longer J5.4 (Pin_4)
- net SPI_MISO: now also J2.2 (Pin_2); no longer J2.4 (Pin_4)
- net SPI_SS: now also J2.4 (Pin_4); no longer J2.2 (Pin_2)
- net TX_PWR_CTRL: now also A1.26 (A7); no longer A1.25 (A6)
Changed lines of the file:
@@
 Wire Notes Line
 	16000 4850 14650 4850
-Text GLabel 15500 4450 0    50   Input ~ 0
+Text GLabel 15500 4250 0    50   Input ~ 0
 Digital_Sensor_CS3
 Text GLabel 15500 4350 0    50   Input ~ 0
 Digital_Sensor_CS2
-Text GLabel 15500 4250 0    50   Input ~ 0
+Text GLabel 15500 4450 0    50   Input ~ 0
 Digital_Sensor_CS1
 Text GLabel 15500 4150 0    50   Input ~ 0
 SPI_SCK
-Text GLabel 15500 4050 0    50   Input ~ 0
+Text GLabel 15500 3850 0    50   Input ~ 0
 SPI_MISO
 Text GLabel 15500 3950 0    50   Input ~ 0
 SPI_MOSI
-Text GLabel 15500 3850 0    50   Input ~ 0
+Text GLabel 15500 4050 0    50   Input ~ 0
 SPI_SS
 Wire Wire Line
@@
 Text Notes 9400 8700 0    50   ~ 0
 REGULATORS
-Text Label 15700 6850 2    50   ~ 0
+Text Label 15700 6750 2    50   ~ 0
 RX_AUDIO
 Text Label 15700 6950 2    50   ~ 0
@@
 Text Label 9350 2550 0    50   ~ 0
 CONTROL_OUTPUT_4
-Text Label 15700 6750 2    50   ~ 0
+Text Label 15700 6850 2    50   ~ 0
 LINK_AUDIO_OUT
 Text Label 15700 6650 2    50   ~ 0
@@
 Text Label 11700 2250 2    50   ~ 0
 LINK_SQUELCH
-Text Label 12700 2650 0    50   ~ 0
+Text Label 12700 2550 0    50   ~ 0
 LINK_PTT_CTRL
 $Comp
@@
 Wire Wire Line
 	1450 9200 1450 9400
-Text Label 650  10350 1    50   ~ 0
+Text Label 4100 10300 1    50   ~ 0
 CONTROL_OUTPUT_0
 Wire Wire Line
@@
 Wire Wire Line
 	4900 9150 4900 9350
-Text Label 4100 10300 1    50   ~ 0
+Text Label 650  10350 1    50   ~ 0
 CONTROL_OUTPUT_2
 Wire Wire Line
@@
 Text Label 4900 7650 2    50   ~ 0
 TX_PWR_CTRL
-Text Label 12700 2550 0    50   ~ 0
+Text Label 12700 2650 0    50   ~ 0
 TX_PWR_CTRL
 Wire Wire Line
